Commit message: 修复wust_arm_driver忘记加载参数的bug，增加线性插值

File: src/wust_arm_7axis_description/urdf/wust_arm_7axis.urdf (robot description, URDF)
Before this commit: robot wust_arm_7axis_description, 15 links, 13 joints
Joints:
- added joint camera_joint: type fixed, parent link7, child camera_link, origin xyz=0.05 0 0.02 rpy=0 0 0
- joint camera_optical_joint: child  -> camera_optical_frame; origin xyz=0 0 0 rpy=0 0 0 -> xyz=0 0 0 rpy=-1.5708 0 -1.5708

Commit message: 新增PLANNING,EXECUTING

File: src/wust_arm_7axis_description/urdf/wust_arm_7axis.urdf (robot description, URDF)
Before this commit: robot wust_arm_7axis_description, 15 links, 14 joints
Joints:
- joint camera_joint: origin xyz=0.05 0 0.02 rpy=0 0 0 -> xyz=0 -0.08 0.04 rpy=0 0 0
- joint camera_optical_joint: origin xyz=0 0 0 rpy=-1.5708 0 -1.5708 -> xyz=0 0 0 rpy=0 0 0
